Commit message: Updated the co-eff of friction in gazebo Updated the paths to files in the .xacro

File: rmp_ros2bot_description/models/urdf/rmp_ros2bot.xacro (robot description, xacro)
@@ -1,7 +1,7 @@
 <?xml version="1.0" ?>
 <robot name="rmp_ros2bot" xmlns:xacro="http://www.ros.org/wiki/xacro">
-<xacro:include filename="$(find rmp_ros2bot_description)/urdf/materials.xacro" />
-<xacro:include filename="$(find rmp_ros2bot_description)/urdf/rmp_ros2bot.trans" />
-<xacro:include filename="$(find rmp_ros2bot_description)/urdf/rmp_ros2bot.gazebo" />
+<xacro:include filename="$(find rmp_ros2bot_description)/models/urdf/materials.xacro" />
+<xacro:include filename="$(find rmp_ros2bot_description)/models/urdf/rmp_ros2bot.trans" />
+<xacro:include filename="$(find rmp_ros2bot_description)/models/urdf/rmp_ros2bot.gazebo" />
 <link name="base_link">
   <inertial>
@@ -13,5 +13,5 @@
     <origin xyz="0 0 0" rpy="0 0 0"/>
     <geometry>
-      <mesh filename="package://rmp_ros2bot_description/meshes/base_link.stl" scale="0.001 0.001 0.001"/>
+      <mesh filename="package://rmp_ros2bot_description/models/meshes/base_link.stl" scale="0.001 0.001 0.001"/>
     </geometry>
     <material name="silver"/>
@@ -20,5 +20,5 @@
     <origin xyz="0 0 0" rpy="0 0 0"/>
     <geometry>
-      <mesh filename="package://rmp_ros2bot_description/meshes/base_link.stl" scale="0.001 0.001 0.001"/>
+      <mesh filename="package://rmp_ros2bot_description/models/meshes/base_link.stl" scale="0.001 0.001 0.001"/>
     </geometry>
   </collision>
@@ -33,5 +33,5 @@
     <origin xyz="0.065 0.085 -0.03" rpy="0 0 0"/>
     <geometry>
-      <mesh filename="package://rmp_ros2bot_description/meshes/right_wheel_1.stl" scale="0.001 0.001 0.001"/>
+      <mesh filename="package://rmp_ros2bot_description/models/meshes/right_wheel_1.stl" scale="0.001 0.001 0.001"/>
     </geometry>
     <material name="silver"/>
@@ -40,5 +40,5 @@
     <origin xyz="0.065 0.085 -0.03" rpy="0 0 0"/>
     <geometry>
-      <mesh filename="package://rmp_ros2bot_description/meshes/right_wheel_1.stl" scale="0.001 0.001 0.001"/>
+      <mesh filename="package://rmp_ros2bot_description/models/meshes/right_wheel_1.stl" scale="0.001 0.001 0.001"/>
     </geometry>
   </collision>
@@ -53,5 +53,5 @@
     <origin xyz="0.065 -0.085 -0.03" rpy="0 0 0"/>
     <geometry>
-      <mesh filename="package://rmp_ros2bot_description/meshes/left_wheel_1.stl" scale="0.001 0.001 0.001"/>
+      <mesh filename="package://rmp_ros2bot_description/models/meshes/left_wheel_1.stl" scale="0.001 0.001 0.001"/>
     </geometry>
     <material name="silver"/>
@@ -60,5 +60,5 @@
     <origin xyz="0.065 -0.085 -0.03" rpy="0 0 0"/>
     <geometry>
-      <mesh filename="package://rmp_ros2bot_description/meshes/left_wheel_1.stl" scale="0.001 0.001 0.001"/>
+      <mesh filename="package://rmp_ros2bot_description/models/meshes/left_wheel_1.stl" scale="0.001 0.001 0.001"/>
     </geometry>
   </collision>
@@ -73,5 +73,5 @@
     <origin xyz="-0.1 -0.0 -0.0175" rpy="0 0 0"/>
     <geometry>
-      <mesh filename="package://rmp_ros2bot_description/meshes/caster_1.stl" scale="0.001 0.001 0.001"/>
+      <mesh filename="package://rmp_ros2bot_description/models/meshes/caster_1.stl" scale="0.001 0.001 0.001"/>
     </geometry>
     <material name="silver"/>
@@ -80,5 +80,5 @@
     <origin xyz="-0.1 -0.0 -0.0175" rpy="0 0 0"/>
     <geometry>
-      <mesh filename="package://rmp_ros2bot_description/meshes/caster_1.stl" scale="0.001 0.001 0.001"/>
+      <mesh filename="package://rmp_ros2bot_description/models/meshes/caster_1.stl" scale="0.001 0.001 0.001"/>
     </geometry>
   </collision>
@@ -93,5 +93,5 @@
     <origin xyz="-0.0 -0.0 -0.0675" rpy="0 0 0"/>
     <geometry>
-      <mesh filename="package://rmp_ros2bot_description/meshes/lidar_1.stl" scale="0.001 0.001 0.001"/>
+      <mesh filename="package://rmp_ros2bot_description/models/meshes/lidar_1.stl" scale="0.001 0.001 0.001"/>
     </geometry>
     <material name="silver"/>
@@ -100,5 +100,5 @@
     <origin xyz="-0.0 -0.0 -0.0675" rpy="0 0 0"/>
     <geometry>
-      <mesh filename="package://rmp_ros2bot_description/meshes/lidar_1.stl" scale="0.001 0.001 0.001"/>
+      <mesh filename="package://rmp_ros2bot_description/models/meshes/lidar_1.stl" scale="0.001 0.001 0.001"/>
     </geometry>
   </collision>
