Commit message: Launch for gazebo working

File: install/rmp_ros2bot_description/share/rmp_ros2bot_description/models/urdf/rmp_ros2bot.xacro (robot description, xacro)
@@ -13,5 +13,5 @@
     <origin xyz="0 0 0" rpy="0 0 0"/>
     <geometry>
-      <mesh filename="package://rmp_ros2bot_description/models/meshes/base_link.stl" scale="0.001 0.001 0.001"/>
+      <mesh filename="file://$(find rmp_ros2bot_description)/models/meshes/base_link.stl" scale="0.001 0.001 0.001"/>
     </geometry>
     <material name="silver"/>
@@ -20,5 +20,5 @@
     <origin xyz="0 0 0" rpy="0 0 0"/>
     <geometry>
-      <mesh filename="package://rmp_ros2bot_description/models/meshes/base_link.stl" scale="0.001 0.001 0.001"/>
+      <mesh filename="file://$(find rmp_ros2bot_description)/models/meshes/base_link.stl" scale="0.001 0.001 0.001"/>
     </geometry>
   </collision>
@@ -33,5 +33,5 @@
     <origin xyz="0.065 0.085 -0.03" rpy="0 0 0"/>
     <geometry>
-      <mesh filename="package://rmp_ros2bot_description/models/meshes/right_wheel_1.stl" scale="0.001 0.001 0.001"/>
+      <mesh filename="file://$(find rmp_ros2bot_description)/models/meshes/right_wheel_1.stl" scale="0.001 0.001 0.001"/>
     </geometry>
     <material name="silver"/>
@@ -40,5 +40,5 @@
     <origin xyz="0.065 0.085 -0.03" rpy="0 0 0"/>
     <geometry>
-      <mesh filename="package://rmp_ros2bot_description/models/meshes/right_wheel_1.stl" scale="0.001 0.001 0.001"/>
+      <mesh filename="file://$(find rmp_ros2bot_description)/models/meshes/right_wheel_1.stl" scale="0.001 0.001 0.001"/>
     </geometry>
   </collision>
@@ -53,5 +53,5 @@
     <origin xyz="0.065 -0.085 -0.03" rpy="0 0 0"/>
     <geometry>
-      <mesh filename="package://rmp_ros2bot_description/models/meshes/left_wheel_1.stl" scale="0.001 0.001 0.001"/>
+      <mesh filename="file://$(find rmp_ros2bot_description)/models/meshes/left_wheel_1.stl" scale="0.001 0.001 0.001"/>
     </geometry>
     <material name="silver"/>
@@ -60,5 +60,5 @@
     <origin xyz="0.065 -0.085 -0.03" rpy="0 0 0"/>
     <geometry>
-      <mesh filename="package://rmp_ros2bot_description/models/meshes/left_wheel_1.stl" scale="0.001 0.001 0.001"/>
+      <mesh filename="file://$(find rmp_ros2bot_description)/models/meshes/left_wheel_1.stl" scale="0.001 0.001 0.001"/>
     </geometry>
   </collision>
@@ -73,5 +73,5 @@
     <origin xyz="-0.1 -0.0 -0.0175" rpy="0 0 0"/>
     <geometry>
-      <mesh filename="package://rmp_ros2bot_description/models/meshes/caster_1.stl" scale="0.001 0.001 0.001"/>
+      <mesh filename="file://$(find rmp_ros2bot_description)/models/meshes/caster_1.stl" scale="0.001 0.001 0.001"/>
     </geometry>
     <material name="silver"/>
@@ -80,5 +80,5 @@
     <origin xyz="-0.1 -0.0 -0.0175" rpy="0 0 0"/>
     <geometry>
-      <mesh filename="package://rmp_ros2bot_description/models/meshes/caster_1.stl" scale="0.001 0.001 0.001"/>
+      <mesh filename="file://$(find rmp_ros2bot_description)/models/meshes/caster_1.stl" scale="0.001 0.001 0.001"/>
     </geometry>
   </collision>
@@ -93,5 +93,5 @@
     <origin xyz="-0.0 -0.0 -0.0675" rpy="0 0 0"/>
     <geometry>
-      <mesh filename="package://rmp_ros2bot_description/models/meshes/lidar_1.stl" scale="0.001 0.001 0.001"/>
+      <mesh filename="file://$(find rmp_ros2bot_description)/models/meshes/lidar_1.stl" scale="0.001 0.001 0.001"/>
     </geometry>
     <material name="silver"/>
@@ -100,5 +100,5 @@
     <origin xyz="-0.0 -0.0 -0.0675" rpy="0 0 0"/>
     <geometry>
-      <mesh filename="package://rmp_ros2bot_description/models/meshes/lidar_1.stl" scale="0.001 0.001 0.001"/>
+      <mesh filename="file://$(find rmp_ros2bot_description)/models/meshes/lidar_1.stl" scale="0.001 0.001 0.001"/>
     </geometry>
   </collision>
