Commit message: Added custom world with robot

File: install/rmp_ros2bot_description/share/rmp_ros2bot_description/models/urdf/materials.xacro (robot description, xacro)
@@ -4,3 +4,6 @@
   <color rgba="0.700 0.700 0.700 1.000"/>
 </material>
+<material name="black">
+  <color rgba="0.0 0.0 0.0 1.000"/>
+</material>
 </robot>

File: install/rmp_ros2bot_description/share/rmp_ros2bot_description/models/urdf/rmp_ros2bot.xacro (robot description, xacro)
@@ -35,5 +35,5 @@
       <mesh filename="file://$(find rmp_ros2bot_description)/models/meshes/right_wheel_1.stl" scale="0.001 0.001 0.001"/>
     </geometry>
-    <material name="silver"/>
+    <material name="black"/>
   </visual>
   <collision>
@@ -55,5 +55,5 @@
       <mesh filename="file://$(find rmp_ros2bot_description)/models/meshes/left_wheel_1.stl" scale="0.001 0.001 0.001"/>
     </geometry>
-    <material name="silver"/>
+    <material name="black"/>
   </visual>
   <collision>

Commit message: Got laser working

File: install/rmp_ros2bot_description/share/rmp_ros2bot_description/models/urdf/materials.xacro (robot description, xacro)
@@ -7,3 +7,6 @@
   <color rgba="0.0 0.0 0.0 1.000"/>
 </material>
+<material name="red">
+  <color rgba="1.0 0.0 0.0 1.000"/>
+</material>
 </robot>

File: install/rmp_ros2bot_description/share/rmp_ros2bot_description/models/urdf/rmp_ros2bot.xacro (robot description, xacro)
@@ -104,4 +104,23 @@
   </collision>
 </link>
+<link name="camera_link">
+    <visual>
+        <geometry>
+            <box size="0.010 0.03 0.03"/>
+        </geometry>
+        <material name="red"/>
+    </visual>
+    <collision>
+    <origin xyz="0.1 0.0 0.0675" rpy="0 0 0"/>
+          <geometry>
+              <box size="0.010 0.03 0.03"/>
+          </geometry>
+      </collision>
+</link>
+<joint name="camera_joint" type="fixed">
+    <parent link="base_link"/>
+    <child link="camera_link"/>
+    <origin xyz="0.1 0.0 0.0675" rpy="0 0 0"/>
+</joint>
 <joint name="right_wheel_joint" type="continuous">
   <origin xyz="-0.065 -0.085 0.03" rpy="0 0 0"/>
